Commit message: resolved depth camera pointlcoud

File: urdf/my_bot.urdf (robot description, URDF)
Before this commit: robot my_bot, 6 links, 5 joints
Links:
- added link camera_link_optical
- link camera_link: geometry visual box size=0.02 0.05 0.05
Joints:
- added joint camera_optical_joint: type fixed, parent camera_link, child camera_link_optical, origin xyz=0 0 0 rpy=${-pi/2} 0 ${-pi/2}
- joint camera_joint: origin xyz=0.1 0 0.075 rpy=0 0 0 -> xyz=0.1 0 0.1 rpy=0 0 0

Commit message: Localization fixed

File: urdf/my_bot.urdf (robot description, URDF)
Before this commit: robot my_bot, 7 links, 6 joints
Links:
- added link gps_link
Joints:
- added joint gps_joint: type fixed, parent base_link, child gps_link, origin xyz=-0.05 0 0.05 rpy=0 0 0
